File: lm386-amp/lm386-amp.sch (KiCad schematic (older format))
At the start: 38 parts

Commit message: Update lm386 amp
Parts:
- removed C?: 470uF, symbol Device:CP
- added C?: 470pF, symbol Device:C
- added R?: 1K, symbol Device:R
- C?: value 470uF -> 220uF
- RV? (x2): value 100K -> 1K
Connections:
- net GND: now also C?.1, R?.1
- net at C?.1, U?.2 (-), U?.3 (+): now also C?.1, C?.2, R?.2; no longer RV?.2
- net at J?.T: now also RV?.1; no longer C?.2
- new net: C?.2, RV?.2
Other:
- note added: "Bridge Mode"
- note removed: "Bidge Mode"
- moved on the sheet: C?, LS?, R?, U?
