File: lm386-amp/lm386-amp.sch (KiCad schematic (older format))
At the start: 39 parts

Commit message: Add some things that have been hanging around
Parts:
- removed C? (x2): 0.1uF, symbol Device:C
- removed C?: 10uF, symbol Device:C
- removed C?: 10uF, symbol Device:CP
- removed C?: 2.2uF, symbol Device:C
- removed C?: 470pF, symbol Device:C
- removed C?: 220uF, symbol Device:CP
- removed C?: 0.033uF, symbol Device:C
- removed J? (x2): AudioJack2, symbol Connector:AudioJack2
- removed LS?: Speaker >=4 Ohms, symbol Device:Speaker
- removed R?: 1K, symbol Device:R
- removed R?: 10R, symbol Device:R
- removed R?: 10K, symbol Device:R
- removed RV? (x2): 1K, symbol Device:R_POT
- removed U?: LM386N-4, symbol Amplifier_Audio:LM386
- added J1: To off-board jack/1K pot assembly, lm386-amp:rs-pro-screw-terminal-block-low-prof-P3.5mm-2x1, symbol Connector:Conn_01x02_Female
- added J2: To power jack/switch assembly, lm386-amp:rs-pro-screw-terminal-block-low-prof-P3.5mm-2x1, symbol Connector:Conn_01x02_Female
- C1: renamed from C?; footprint (none) -> Capacitor_THT:CP_Radial_D5.0mm_P2.50mm
- C10, C5: renamed from C?; footprint (none) -> Capacitor_THT:C_Disc_D4.7mm_W2.5mm_P5.00mm
- C11, C4, C6, C9: renamed from C?; footprint (none) -> Capacitor_THT:CP_Radial_D6.3mm_P2.50mm
- C12, C2, C3, C7, C8: renamed from C?; footprint (none) -> Capacitor_THT:C_Disc_D3.4mm_W2.1mm_P2.50mm
- C13: renamed from C?; footprint (none) -> Capacitor_THT:CP_Radial_D8.0mm_P2.50mm
- LS1: renamed from LS?; footprint (none) -> lm386-amp:rs-pro-screw-terminal-block-low-prof-P3.5mm-2x1
- R1: renamed from R?; footprint (none) -> Resistor_THT:R_Axial_DIN0411_L9.9mm_D3.6mm_P12.70mm_Horizontal
- R2, R4: renamed from R?; value 1K -> 1K (0.1%); footprint (none) -> Resistor_THT:R_Axial_DIN0411_L9.9mm_D3.6mm_P12.70mm_Horizontal
- R3, R5, R6: renamed from R?; footprint (none) -> Resistor_THT:R_Axial_DIN0204_L3.6mm_D1.6mm_P7.62mm_Horizontal
- U1, U2: renamed from U?; footprint (none) -> Package_DIP:DIP-8_W7.62mm_Socket
Connections:
- net +12V: now also J2.2 (Pin_2)
- net GND: now also J1.1 (Pin_1), J2.1 (Pin_1)
- net at C1.2: now also J1.2 (Pin_2)
Other:
- note removed: "Bass boost"
- note removed: "Bridge Mode"
- note removed: "Gain control"
- note removed: "Power supply decoupling"
- note removed: "Standard Mode"
- moved on the sheet: C1, C10, C11, C12, C13, C2, C3, C4, C5, C6, C7, C8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
